File: usb_c_cable_tester_tester/usb_c_cable_tester_tester.kicad_pcb (KiCad board)
At the start: 2 copper layers, 100 x 50 mm, 10 parts, among them SW1 SW_DIP_x04, SW2 SW_DIP_x08, SW3 SW_DIP_x08, SW4 SW_DIP_x05

Commit message: layout finished
Parts:
- added kibuzzard-678D5650: G***, kibuzzard-678D5650, F.Cu at (115.2, 115.1)
- added kibuzzard-678D569F: G***, kibuzzard-678D569F, F.Cu at (147.6, 115.1)
- added kibuzzard-678D56BE: G***, kibuzzard-678D56BE, F.Cu at (145.1, 115.1)
- added kibuzzard-678D56C4: G***, kibuzzard-678D56C4, F.Cu at (180.0, 115.1)
- added kibuzzard-678D56CC: G***, kibuzzard-678D56CC, F.Cu at (142.5, 115.1)
- added kibuzzard-678D56D1: G***, kibuzzard-678D56D1, F.Cu at (140.0, 115.1)
- added kibuzzard-678D56D6: G***, kibuzzard-678D56D6, F.Cu at (137.5, 115.1)
- added kibuzzard-678D56DC: G***, kibuzzard-678D56DC, F.Cu at (134.9, 115.1)
- added kibuzzard-678D56E1: G***, kibuzzard-678D56E1, F.Cu at (182.6, 115.1)
- added kibuzzard-678D56E7: G***, kibuzzard-678D56E7, F.Cu at (132.4, 115.1)
- added kibuzzard-678D56EC: G***, kibuzzard-678D56EC, F.Cu at (129.8, 115.1)
- added kibuzzard-678D56F1: G***, kibuzzard-678D56F1, F.Cu at (112.7, 115.1)
- added kibuzzard-678D5711: G***, kibuzzard-678D5711, F.Cu at (117.8, 115.1)
- added kibuzzard-678D5716: G***, kibuzzard-678D5716, F.Cu at (155.2, 115.1)
- added kibuzzard-678D571B: G***, kibuzzard-678D571B, F.Cu at (157.8, 115.1)
- added kibuzzard-678D5720: G***, kibuzzard-678D5720, F.Cu at (185.1, 115.1)
- added kibuzzard-678D5725: G***, kibuzzard-678D5725, F.Cu at (160.3, 115.1)
- added kibuzzard-678D572A: G***, kibuzzard-678D572A, F.Cu at (162.9, 115.1)
- added kibuzzard-678D572F: G***, kibuzzard-678D572F, F.Cu at (165.4, 115.1)
- added kibuzzard-678D5733: G***, kibuzzard-678D5733, F.Cu at (167.9, 115.1)
- added kibuzzard-678D5738: G***, kibuzzard-678D5738, F.Cu at (187.6, 115.1)
- added kibuzzard-678D573D: G***, kibuzzard-678D573D, F.Cu at (170.5, 115.1)
- added kibuzzard-678D5742: G***, kibuzzard-678D5742, F.Cu at (173.0, 115.1)
- added kibuzzard-678D5747: G***, kibuzzard-678D5747, F.Cu at (120.3, 115.1)
- added kibuzzard-678D5F38: G***, kibuzzard-678D5F38, F.Cu at (120.3, 135.4)
- added kibuzzard-678D5F38: G***, kibuzzard-678D5F38, F.Cu at (112.7, 135.4)
- added kibuzzard-678D5F38: G***, kibuzzard-678D5F38, F.Cu at (117.8, 135.4)
- added kibuzzard-678D5F38: G***, kibuzzard-678D5F38, F.Cu at (115.2, 135.4)
- added kibuzzard-678D5FA3: G***, kibuzzard-678D5FA3, F.Cu at (122.9, 135.4)
- added kibuzzard-678D5FC4: G***, kibuzzard-678D5FC4, F.Cu at (129.8, 136.0)
- added kibuzzard-678D5FDE: G***, kibuzzard-678D5FDE, F.Cu at (132.4, 136.0)
- added kibuzzard-678D5FEA: G***, kibuzzard-678D5FEA, F.Cu at (187.6, 136.0)
- added kibuzzard-678D5FEA: G***, kibuzzard-678D5FEA, F.Cu at (180.0, 136.0)
- added kibuzzard-678D5FEA: G***, kibuzzard-678D5FEA, F.Cu at (185.1, 136.0)
- added kibuzzard-678D5FEA: G***, kibuzzard-678D5FEA, F.Cu at (182.6, 136.0)
- added kibuzzard-678D6F6F: G***, kibuzzard-678D6F6F, F.Cu at (134.9, 136.0)
- added kibuzzard-678D6F82: G***, kibuzzard-678D6F82, F.Cu at (137.5, 136.0)
- added kibuzzard-678D6F8E: G***, kibuzzard-678D6F8E, F.Cu at (140.0, 136.0)
- added kibuzzard-678D6F9D: G***, kibuzzard-678D6F9D, F.Cu at (142.5, 136.0)
- added kibuzzard-678D6FAB: G***, kibuzzard-678D6FAB, F.Cu at (145.1, 136.0)
- added kibuzzard-678D6FB9: G***, kibuzzard-678D6FB9, F.Cu at (147.6, 136.0)
- added kibuzzard-678D6FD7: G***, kibuzzard-678D6FD7, F.Cu at (155.2, 136.0)
- added kibuzzard-678D6FE6: G***, kibuzzard-678D6FE6, F.Cu at (157.8, 136.0)
- added kibuzzard-678D700A: G***, kibuzzard-678D700A, F.Cu at (160.3, 136.0)
- added kibuzzard-678D7016: G***, kibuzzard-678D7016, F.Cu at (162.9, 136.0)
- added kibuzzard-678D7021: G***, kibuzzard-678D7021, F.Cu at (165.4, 136.0)
- added kibuzzard-678D7031: G***, kibuzzard-678D7031, F.Cu at (167.9, 136.0)
- added kibuzzard-678D7040: G***, kibuzzard-678D7040, F.Cu at (170.5, 136.0)
- added kibuzzard-678D704B: G***, kibuzzard-678D704B, F.Cu at (173.0, 136.0)
Connections:
- SW2 pad 10: Net-(USB2-SSRXn1) -> Net-(USB2-SSTXn2)
- SW2 pad 11: Net-(USB2-SUB2) -> Net-(USB2-CC2)
- SW2 pad 12: Net-(USB2-DN2) -> Net-(USB2-DP2)
- SW2 pad 13: Net-(USB2-DP2) -> Net-(USB2-DN2)
- SW2 pad 14: Net-(USB2-CC2) -> Net-(USB2-SUB2)
- SW2 pad 15: Net-(USB2-SSTXn2) -> Net-(USB2-SSRXn1)
- SW2 pad 16: Net-(USB2-SSTXp2) -> Net-(USB2-SSRXp1)
- SW2 pad 9: Net-(USB2-SSRXp1) -> Net-(USB2-SSTXp2)
- USB2 pad B1: Net-(SW4-Pad10) -> Net-(SW4-Pad9)
- USB2 pad B12: Net-(SW4-Pad9) -> Net-(SW4-Pad10)
- USB2 pad B4: Net-(SW1-Pad8) -> Net-(SW1-Pad7)
- USB2 pad B9: Net-(SW1-Pad7) -> Net-(SW1-Pad8)
Routing:
- net Net-(USB2-SSTXp2): track 88.9 -> 71.1 mm
- net Net-(USB2-SSRXp1): track 77.7 -> 92.9 mm, vias 2 -> 3
- net Net-(USB2-SSTXn2): track 85.2 -> 72.5 mm
- net Net-(USB2-SSRXn1): track 79.2 -> 88.2 mm, vias 2 -> 3
- net Net-(USB2-CC2): track 87.9 -> 80.3 mm
- net Net-(SW1-Pad7): track 39.3 -> 32.8 mm
- net Net-(SW4-Pad10): track 105.1 -> 111.0 mm
- net Net-(SW4-Pad9): track 109.9 -> 104.5 mm
- net Net-(SW1-Pad8): track 35.3 -> 39.7 mm, vias 2 -> 0
- net Net-(USB2-DN2): track 81.3 -> 78.4 mm, vias 2 -> 3
- net Net-(USB2-SUB2): track 87.3 -> 90.2 mm, vias 2 -> 3
- net Net-(USB2-DP2): track 76.5 -> 73.9 mm
Other:
- board text added: "USB-C-Cable-Tester-Tester @casartar 2025 v1.0"
