File: usb_c_cable_tester_tester/usb_c_cable_tester_tester.kicad_sch (KiCad schematic)
At the start: 6 parts, among them J1 USB_C_Receptacle, J2 USB_C_Receptacle, SW1 SW_DIP_x04, SW2 SW_DIP_x08, SW3 SW_DIP_x08, SW4 SW_DIP_x05

Commit message: first layout
Parts:
- removed J1, J2: USB_C_Receptacle, easyeda:USB-C-SMD_UT11113-11602-7H, symbol Connector:USB_C_Receptacle
- added H1, H2, H3, H4: MountingHole, MountingHole:MountingHole_3.2mm_M3, symbol Mechanical:MountingHole
- added USB1, USB2: UT11113-11602-7H, easyeda2kicad:USB-C-SMD_UT11113-11602-7H, symbol easyeda2kicad:UT11113-11602-7H
- SW1: footprint (none) -> Button_Switch_THT:SW_DIP_SPSTx04_Slide_9.78x12.34mm_W7.62mm_P2.54mm
- SW2, SW3: footprint (none) -> Button_Switch_THT:SW_DIP_SPSTx08_Slide_9.78x22.5mm_W7.62mm_P2.54mm
- SW4: footprint (none) -> Button_Switch_THT:SW_DIP_SPSTx05_Slide_9.78x14.88mm_W7.62mm_P2.54mm
Connections:
- net at SW4.7: now also USB2.A12 (GND)
- net at SW3.14: now also USB2.A5 (CC1)
- net at SW3.13: now also USB2.A6 (DP1)
- net at SW4.8: now also USB2.A1 (GND)
- net at SW3.15: now also USB2.A3 (SSTXn1)
- net at SW3.16: now also USB2.A2 (SSTXP1)
- net at SW1.8: now also USB2.B4 (VBUS)
- net at SW2.16: now also USB2.B2 (SSTXp2)
- net at SW2.12: now also USB2.B7 (DN2)
- net at SW2.14: now also USB2.B5 (CC2)
- net at SW3.10: now also USB2.A10 (SSRXn2)
- net at SW1.7: now also USB2.B9 (VBUS)
- net at SW4.9: now also USB2.B12 (GND)
- net at SW2.10: now also USB2.B10 (SSRXn1)
- net at SW2.9: now also USB2.B11 (SSRXp1)
- net at SW4.10: now also USB2.B1 (GND)
- net at SW3.11: now also USB2.A8 (SUB1)
- net at SW3.12: now also USB2.A7 (DN1)
- net at SW1.5: now also USB2.A9 (VBUS)
- net at SW2.15: now also USB2.B3 (SSTXn2)
- net at SW2.11: now also USB2.B8 (SUB2)
- net at SW2.13: now also USB2.B6 (DP2)
- net at SW3.9: now also USB2.A11 (SSRXp2)
- net at SW1.6: now also USB2.A4 (VBUS)
- net at SW4.6: now also USB2.25 (EH), USB2.26 (EH), USB2.27 (EH), USB2.28 (EH), USB2.29 (EH), USB2.30 (EH)
- net at SW2.1: now also USB1.B11 (SSRXp1)
- net at SW2.2: now also USB1.B10 (SSRXn1)
- net at SW2.3: now also USB1.B8 (SUB2)
- net at SW2.4: now also USB1.B7 (DN2)
- net at SW2.5: now also USB1.B6 (DP2)
- net at SW2.6: now also USB1.B5 (CC2)
- net at SW2.7: now also USB1.B3 (SSTXn2)
- net at SW2.8: now also USB1.B2 (SSTXp2)
- net at SW4.4: now also USB1.A12 (GND)
- net at SW3.3: now also USB1.A5 (CC1)
- net at SW3.4: now also USB1.A6 (DP1)
- net at SW4.3: now also USB1.A1 (GND)
- net at SW3.2: now also USB1.A3 (SSTXn1)
- net at SW3.1: now also USB1.A2 (SSTXP1)
- net at SW1.1: now also USB1.B9 (VBUS)
- net at SW3.7: now also USB1.A10 (SSRXn2)
- net at SW1.2: now also USB1.B4 (VBUS)
- net at SW4.2: now also USB1.B1 (GND)
- net at SW4.1: now also USB1.B12 (GND)
- net at SW3.6: now also USB1.A8 (SUB1)
- net at SW3.5: now also USB1.A7 (DN1)
- net at SW1.4: now also USB1.A9 (VBUS)
- net at SW3.8: now also USB1.A11 (SSRXp2)
- net at SW1.3: now also USB1.A4 (VBUS)
- net at SW4.5: now also USB1.25 (EH), USB1.26 (EH), USB1.27 (EH), USB1.28 (EH), USB1.29 (EH), USB1.30 (EH)

Commit message: layout finished
Connections:
- net at SW4.10: now also USB2.B12 (GND); no longer USB2.B1 (GND)
- net at SW4.9: now also USB2.B1 (GND); no longer USB2.B12 (GND)
- net at USB2.B10 (SSRXn1): now also SW2.15; no longer SW2.10
- net at USB2.B11 (SSRXp1): now also SW2.16; no longer SW2.9
- net at USB2.B2 (SSTXp2): now also SW2.9; no longer SW2.16
- net at USB2.B3 (SSTXn2): now also SW2.10; no longer SW2.15
- net at USB2.B4 (VBUS): now also SW1.7; no longer SW1.8
- net at USB2.B5 (CC2): now also SW2.11; no longer SW2.14
- net at USB2.B6 (DP2): now also SW2.12; no longer SW2.13
- net at USB2.B7 (DN2): now also SW2.13; no longer SW2.12
- net at USB2.B8 (SUB2): now also SW2.14; no longer SW2.11
- net at USB2.B9 (VBUS): now also SW1.8; no longer SW1.7
Changed lines of the file:
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@@
+	(wire
+		(pts
+			(xy 182.88 226.06) (xy 182.88 210.82)
+		)
+		(stroke
+			(width 0)
+			(type default)
+		)
+	)
 	(wire
 		(pts
@@
 	(wire
 		(pts
-			(xy 210.82 208.28) (xy 210.82 226.06)
-		)
-		(stroke
-			(width 0)
-			(type default)
-		)
-	)
-	(wire
-		(pts
 			(xy 232.41 261.62) (xy 229.87 261.62)
 		)
@@
 	(wire
 		(pts
-			(xy 217.17 246.38) (xy 190.5 246.38)
-		)
-		(stroke
-			(width 0)
-			(type default)
-		)
-	)
-	(wire
-		(pts
 			(xy 266.7 238.76) (xy 266.7 187.96)
 		)
@@
 	(wire
 		(pts
-			(xy 193.04 243.84) (xy 193.04 160.02)
+			(xy 193.04 160.02) (xy 193.04 236.22)
 		)
 		(stroke
@@
 	(wire
 		(pts
+			(xy 205.74 248.92) (xy 217.17 248.92)
+		)
+		(stroke
+			(width 0)
+			(type default)
+		)
+	)
+	(wire
+		(pts
 			(xy 113.03 111.76) (xy 124.46 111.76)
 		)
@@
 	(wire
 		(pts
-			(xy 217.17 254) (xy 182.88 254)
-		)
-		(stroke
-			(width 0)
-			(type default)
-		)
-	)
-	(wire
-		(pts
 			(xy 113.03 101.6) (xy 134.62 101.6)
 		)
@@
 	(wire
 		(pts
-			(xy 203.2 127) (xy 203.2 233.68)
-		)
-		(stroke
-			(width 0)
-			(type default)
-		)
-	)
-	(wire
-		(pts
 			(xy 157.48 190.5) (xy 137.16 190.5)
 		)
@@
 	(wire
 		(pts
+			(xy 200.66 243.84) (xy 217.17 243.84)
+		)
+		(stroke
+			(width 0)
+			(type default)
+		)
+	)
+	(wire
+		(pts
 			(xy 157.48 132.08) (xy 127 132.08)
 		)
@@
 	(wire
 		(pts
-			(xy 217.17 238.76) (xy 198.12 238.76)
-		)
-		(stroke
-			(width 0)
-			(type default)
-		)
-	)
-	(wire
-		(pts
 			(xy 279.4 251.46) (xy 279.4 177.8)
 		)
@@
 	(wire
 		(pts
-			(xy 190.5 246.38) (xy 190.5 129.54)
+			(xy 190.5 129.54) (xy 190.5 233.68)
 		)
 		(stroke
@@
 	(wire
 		(pts
-			(xy 217.17 231.14) (xy 205.74 231.14)
-		)
-		(stroke
-			(width 0)
-			(type default)
-		)
-	)
-	(wire
-		(pts
 			(xy 113.03 96.52) (xy 139.7 96.52)
 		)
@@
 	(wire
 		(pts
+			(xy 210.82 254) (xy 217.17 254)
+		)
+		(stroke
+			(width 0)
+			(type default)
+		)
+	)
+	(wire
+		(pts
 			(xy 113.03 106.68) (xy 129.54 106.68)
 		)
@@
 	(wire
 		(pts
-			(xy 217.17 248.92) (xy 187.96 248.92)
-		)
-		(stroke
-			(width 0)
-			(type default)
-		)
-	)
-	(wire
-		(pts
 			(xy 55.88 96.52) (xy 82.55 96.52)
 		)
@@
 	(wire
 		(pts
+			(xy 193.04 236.22) (xy 217.17 236.22)
+		)
+		(stroke
+			(width 0)
+			(type default)
+		)
+	)
+	(wire
+		(pts
 			(xy 274.32 132.08) (xy 172.72 132.08)
 		)
@@
 	(wire
 		(pts
-			(xy 200.66 236.22) (xy 200.66 152.4)
+			(xy 200.66 152.4) (xy 200.66 243.84)
 		)
 		(stroke
@@
 	(wire
 		(pts
+			(xy 208.28 251.46) (xy 217.17 251.46)
+		)
+		(stroke
+			(width 0)
+			(type default)
+		)
+	)
+	(wire
+		(pts
 			(xy 157.48 180.34) (xy 124.46 180.34)
 		)
@@
 	(wire
 		(pts
-			(xy 182.88 254) (xy 182.88 210.82)
-		)
-		(stroke
-			(width 0)
-			(type default)
-		)
-	)
-	(wire
-		(pts
 			(xy 195.58 157.48) (xy 172.72 157.48)
 		)
@@
 	(wire
 		(pts
-			(xy 217.17 241.3) (xy 195.58 241.3)
+			(xy 210.82 254) (xy 210.82 208.28)
+		)
+		(stroke
+			(width 0)
+			(type default)
+		)
+	)
+	(wire
+		(pts
+			(xy 190.5 233.68) (xy 217.17 233.68)
 		)
 		(stroke
@@
 	(wire
 		(pts
-			(xy 217.17 243.84) (xy 193.04 243.84)
-		)
-		(stroke
-			(width 0)
-			(type default)
-		)
-	)
-	(wire
-		(pts
 			(xy 60.96 101.6) (xy 82.55 101.6)
 		)
@@
 	(wire
 		(pts
-			(xy 185.42 251.46) (xy 185.42 165.1)
+			(xy 185.42 165.1) (xy 185.42 228.6)
 		)
 		(stroke
@@
 	(wire
 		(pts
-			(xy 217.17 228.6) (xy 208.28 228.6)
-		)
-		(stroke
-			(width 0)
-			(type default)
-		)
-	)
-	(wire
-		(pts
-			(xy 217.17 236.22) (xy 200.66 236.22)
-		)
-		(stroke
-			(width 0)
-			(type default)
-		)
-	)
-	(wire
-		(pts
-			(xy 187.96 248.92) (xy 187.96 162.56)
+			(xy 203.2 246.38) (xy 217.17 246.38)
+		)
+		(stroke
+			(width 0)
+			(type default)
+		)
+	)
+	(wire
+		(pts
+			(xy 187.96 162.56) (xy 187.96 231.14)
 		)
 		(stroke
@@
 	(wire
 		(pts
+			(xy 205.74 149.86) (xy 205.74 248.92)
+		)
+		(stroke
+			(width 0)
+			(type default)
+		)
+	)
+	(wire
+		(pts
 			(xy 63.5 154.94) (xy 63.5 104.14)
 		)
@@
 	(wire
 		(pts
+			(xy 198.12 241.3) (xy 217.17 241.3)
+		)
+		(stroke
+			(width 0)
+			(type default)
+		)
+	)
+	(wire
+		(pts
+			(xy 187.96 231.14) (xy 217.17 231.14)
+		)
+		(stroke
+			(width 0)
+			(type default)
+		)
+	)
+	(wire
+		(pts
+			(xy 203.2 127) (xy 203.2 246.38)
+		)
+		(stroke
+			(width 0)
+			(type default)
+		)
+	)
+	(wire
+		(pts
 			(xy 157.48 215.9) (xy 147.32 215.9)
 		)
@@
 	(wire
 		(pts
-			(xy 205.74 149.86) (xy 205.74 231.14)
-		)
-		(stroke
-			(width 0)
-			(type default)
-		)
-	)
-	(wire
-		(pts
 			(xy 113.03 91.44) (xy 144.78 91.44)
 		)
@@
 	(wire
 		(pts
-			(xy 217.17 226.06) (xy 210.82 226.06)
-		)
-		(stroke
-			(width 0)
-			(type default)
-		)
-	)
-	(wire
-		(pts
 			(xy 48.26 210.82) (xy 48.26 88.9)
 		)
@@
 	(wire
 		(pts
+			(xy 185.42 228.6) (xy 217.17 228.6)
+		)
+		(stroke
+			(width 0)
+			(type default)
+		)
+	)
+	(wire
+		(pts
 			(xy 113.03 109.22) (xy 127 109.22)
 		)
@@
 	(wire
 		(pts
-			(xy 198.12 238.76) (xy 198.12 154.94)
-		)
-		(stroke
-			(width 0)
-			(type default)
-		)
-	)
-	(wire
-		(pts
-			(xy 217.17 233.68) (xy 203.2 233.68)
+			(xy 198.12 154.94) (xy 198.12 241.3)
 		)
 		(stroke
@@
 	(wire
 		(pts
-			(xy 208.28 147.32) (xy 208.28 228.6)
+			(xy 182.88 226.06) (xy 217.17 226.06)
+		)
+		(stroke
+			(width 0)
+			(type default)
+		)
+	)
+	(wire
+		(pts
+			(xy 208.28 147.32) (xy 208.28 251.46)
 		)
 		(stroke
@@
 	(wire
 		(pts
+			(xy 195.58 238.76) (xy 217.17 238.76)
+		)
+		(stroke
+			(width 0)
+			(type default)
+		)
+	)
+	(wire
+		(pts
 			(xy 66.04 106.68) (xy 82.55 106.68)
 		)
@@
 	(wire
 		(pts
-			(xy 217.17 251.46) (xy 185.42 251.46)
-		)
-		(stroke
-			(width 0)
-			(type default)
-		)
-	)
-	(wire
-		(pts
-			(xy 195.58 241.3) (xy 195.58 157.48)
-		)
-		(stroke
+			(xy 195.58 157.48) (xy 195.58 238.76)
+		)
+		(stroke
